File: keyvas.kicad_sch (KiCad schematic)
At the start: 113 parts, among them J2 SWD, J3 USB-C Conn, J4 Conn_01x02_Female, K1 KEYSW, K10 KEYSW, K11 KEYSW, K12 KEYSW, K13 KEYSW, K14 KEYSW, K15 KEYSW, K16 KEYSW, K17 KEYSW, K18 KEYSW, K19 KEYSW, K2 KEYSW, K20 KEYSW, K21 KEYSW, K22 KEYSW, K23 KEYSW, K24 KEYSW, K25 KEYSW, K26 KEYSW, K27 KEYSW, K28 KEYSW, K29 KEYSW, K3 KEYSW, K30 KEYSW, K31 KEYSW, K32 KEYSW, K33 KEYSW, K34 KEYSW, K35 KEYSW, K36 KEYSW, K37 KEYSW, K38 KEYSW, K39 KEYSW, K4 KEYSW, K40 KEYSW, K5 KEYSW, K6 KEYSW, K7 KEYSW, K8 KEYSW, K9 KEYSW, Q2 AO3407, SW31 SW_SPDT, U2 XC6220B331MR-G, U3 TP4054, U4 USBLC6-2SC6, U5 E73-2G4M08S1C

Commit message: scheme
Parts:
- added D44, D45, D46, D47, D48, D49, D50, D51: D_Small, kbd:D3_SMD, symbol Device:D_Small
- added K41, K42, K43, K44, K45, K46, K47, K48: KEYSW, kbd:keyswitch_gateron_low_profile_1u, symbol Keyboard_Components:KEYSW
- added X1: 32.768kHz, kbd:Crystal_SMD_MicroCrystal_CM9V-T1A-2Pin_1.6x1.0mm_HandSoldering_REV, symbol Device:Crystal_Small
- K1: footprint kbd:ChocV1_V2_Hotswap -> kbd:keyswitch_gateron_low_profile_1u
- K10, K11, K12, K13, K14, K15, K16, K17, K18, K19, K2, K20, K21, K22, K23, K24, K25, K26, K27, K28, K29, K3, K30, K31, K32, K33, K34, K35, K36, K37, K38, K39, K4, K40, K5, K6, K7, K8, K9: footprint kbd:MX-Alps-1U-REV -> kbd:keyswitch_gateron_low_profile_1u
Connections:
- net BATTERY_PIN: now also U5.7 (P0.02/AIN0*)
- net BLUE_LED: now also U5.2 (P1.10*)
- net COL0: now also K13.2 (B), K25.2 (B), K37.2 (B), U5.10 (P0.30/AIN6*); no longer K11.2 (B), K21.2 (B)
- net COL1: now also K14.2 (B), K26.2 (B), K38.2 (B), U5.9 (P0.31/AIN7*); no longer K12.2 (B), K22.2 (B)
- net COL2: now also K15.2 (B), K27.2 (B), K39.2 (B), U5.8 (P0.29/AIN5*); no longer K13.2 (B), K23.2 (B)
- net COL3: now also K16.2 (B), K28.2 (B), K40.2 (B), U5.6 (P1.13*); no longer K14.2 (B), K24.2 (B)
- net COL4: now also K17.2 (B), K29.2 (B), U5.4 (P0.28/AIN4*), K41.2 (B); no longer K15.2 (B), K25.2 (B)
- net COL5: now also K18.2 (B), K30.2 (B), U5.3 (P0.03/AIN1*), K42.2 (B); no longer K16.2 (B), K26.2 (B)
- net COL6: now also K19.2 (B), K31.2 (B), U5.1 (P1.11*), K43.2 (B); no longer K17.2 (B), K27.2 (B)
- net COL7: now also K20.2 (B), K32.2 (B), U5.22 (P0.07), K44.2 (B); no longer K18.2 (B), K28.2 (B)
- net COL8: now also K21.2 (B), K33.2 (B), U5.20 (P0.12), K45.2 (B); no longer K19.2 (B), K29.2 (B), K39.2 (B)
- net COL9: now also K22.2 (B), K34.2 (B), U5.18 (P0.04/AIN2), K46.2 (B); no longer K20.2 (B), K30.2 (B), K40.2 (B)
- net DATA+: now also U5.31 (D+)
- net DATA-: now also U5.29 (D-)
- net GND: now also U5.21 (GND), U5.24 (GND), U5.5 (GND)
- net ROW0: now also D11.1 (K), D12.1 (K), U5.12 (P0.26)
- net ROW1: now also D21.1 (K), D22.1 (K), D23.1 (K), D24.1 (K), U5.28 (P0.15); no longer D11.1 (K), D12.1 (K)
- net ROW2: now also D32.1 (K), D33.1 (K), D34.1 (K), D37.1 (K), D38.1 (K), D39.1 (K), U5.30 (P0.17); no longer D21.1 (K), D22.1 (K), D23.1 (K), D24.1 (K)
- net ROW3: now also U5.32 (P0.20), D44.1 (K), D45.1 (K), D46.1 (K), D47.1 (K), D48.1 (K), D49.1 (K), D50.1 (K), D51.1 (K); no longer D32.1 (K), D33.1 (K), D34.1 (K), D37.1 (K), D38.1 (K), D39.1 (K)
- net SWC: now also U5.39 (SWDCLK)
- net SWD: now also U5.37 (SWDIO)
- net VBUS: now also U5.27 (VBUS)
- net nRF_VDD: now also U5.19 (VDD), U5.23 (VDDH)
- net COL10: now reaches K35.2 (B)
- net COL10: now also K11.2 (B), K23.2 (B), U5.16 (P0.08), K47.2 (B)
- net at U5.11 (P0.00/XL1): now also X1.2
- net at U5.13 (P0.01/XL2): now also X1.1
- net COL11: now reaches U5.14 (P0.06)
- net COL11: now also K12.2 (B), K24.2 (B), K36.2 (B), K48.2 (B)
- net PROG: now reaches U5.15 (P0.05/AIN3)
- new net: D51.2 (A), K48.1 (A)
- new net: D45.2 (A), K42.1 (A)
- new net: D48.2 (A), K45.1 (A)
- new net: D49.2 (A), K46.1 (A)
- new net: D46.2 (A), K43.1 (A)
- new net: D47.2 (A), K44.1 (A)
- new net: D44.2 (A), K41.1 (A)
- new net: D50.2 (A), K47.1 (A)
Other:
- moved on the sheet: C1, C2, C3, C4, C5, D1, D31, D35, D36, F1, H1, H3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
