File: keyvas.kicad_sch (KiCad schematic)
At the start: 130 parts, among them J2 SWD, J3 USB-C Conn, J4 Conn_01x02_Female, K1 KEYSW, K10 KEYSW, K11 KEYSW, K12 KEYSW, K13 KEYSW, K14 KEYSW, K15 KEYSW, K16 KEYSW, K17 KEYSW, K18 KEYSW, K19 KEYSW, K2 KEYSW, K20 KEYSW, K21 KEYSW, K22 KEYSW, K23 KEYSW, K24 KEYSW, K25 KEYSW, K26 KEYSW, K27 KEYSW, K28 KEYSW, K29 KEYSW, K3 KEYSW, K30 KEYSW, K31 KEYSW, K32 KEYSW, K33 KEYSW, K34 KEYSW, K35 KEYSW, K36 KEYSW, K37 KEYSW, K38 KEYSW, K39 KEYSW, K4 KEYSW, K40 KEYSW, K41 KEYSW, K42 KEYSW, K43 KEYSW, K44 KEYSW, K45 KEYSW, K46 KEYSW, K47 KEYSW, K48 KEYSW, K5 KEYSW, K6 KEYSW, K7 KEYSW, K8 KEYSW, K9 KEYSW, Q2 AO3407, SW31 SW_SPDT, U2 XC6220B331MR-G, U3 TP4054, U4 USBLC6-2SC6, U5 E73-2G4M08S1C, X1 32.768kHz

Commit message: Продолжаем натягивать сову на глобус
Parts:
- K1, K10, K11, K12, K13, K14, K15, K16, K17, K18, K19, K2, K20, K21, K22, K23, K24, K25, K26, K27, K28, K29, K3, K30, K31, K32, K33, K34, K35, K36, K37, K38, K39, K4, K40, K41, K42, K43, K44, K45, K46, K47, K48, K5, K6, K7, K8, K9: footprint kbd:keyswitch_gateron_low_profile_1u -> kbd:keyswitch_NumPy_gateon_cherry
Connections:
- net ROW0: now also U5.43 (P0.10/NFC2*); no longer U5.12 (P0.26)
- net ROW2: now also U5.33 (P0.13); no longer U5.30 (P0.17)
- net ROW3: now also U5.35 (P0.24); no longer U5.32 (P0.20)
Changed lines of the file:
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@@
 	(wire
 		(pts
+			(xy 26.67 58.42) (xy 27.94 58.42)
+		)
+		(stroke
+			(width 0)
+			(type default)
+		)
+	)
+	(wire
+		(pts
 			(xy 163.83 127) (xy 163.83 142.24)
 		)
@@
 	(wire
 		(pts
+			(xy 26.67 62.23) (xy 27.94 62.23)
+		)
+		(stroke
+			(width 0)
+			(type default)
+		)
+	)
+	(wire
+		(pts
 			(xy 106.68 109.22) (xy 106.68 111.76)
 		)
@@
 	(wire
 		(pts
+			(xy 27.94 77.47) (xy 26.67 77.47)
+		)
+		(stroke
+			(width 0)
+			(type default)
+		)
+	)
+	(wire
+		(pts
 			(xy 119.38 149.86) (xy 130.81 149.86)
 		)
@@
 	(global_label "ROW0"
 		(shape input)
-		(at 77.47 86.36 270)
+		(at 26.67 77.47 180)
 		(effects
 			(font
@@
 		)
 		(property "Intersheetrefs" "${INTERSHEET_REFS}"
-			(at 77.3906 95.5585 90)
+			(at 17.4715 77.3906 0)
 			(effects
 				(font
@@
 	(global_label "ROW3"
 		(shape input)
-		(at 66.04 86.36 270)
+		(at 26.67 62.23 180)
 		(fields_autoplaced yes)
 		(effects
@@
 		)
 		(property "Intersheetrefs" "${INTERSHEET_REFS}"
-			(at 66.04 94.6066 90)
+			(at 18.4234 62.23 0)
 			(effects
 				(font
@@
 	(global_label "ROW2"
 		(shape input)
-		(at 69.85 86.36 270)
+		(at 26.67 58.42 180)
 		(effects
 			(font
@@
 		)
 		(property "Intersheetrefs" "${INTERSHEET_REFS}"
-			(at 69.7706 95.5585 90)
+			(at 17.4715 58.3406 0)
 			(effects
 				(font
@@
 			)
 		)
-		(property "Footprint" "kbd:keyswitch_gateron_low_profile_1u"
+		(property "Footprint" "kbd:keyswitch_NumPy_gateon_cherry"
 			(at 158.75 152.4 0)
 			(effects
@@
 			)
 		)
-		(property "Footprint" "kbd:keyswitch_gateron_low_profile_1u"
+		(property "Footprint" "kbd:keyswitch_NumPy_gateon_cherry"
 			(at 55.88 106.68 0)
 			(effects
@@
 			)
 		)
-		(property "Footprint" "kbd:keyswitch_gateron_low_profile_1u"
+		(property "Footprint" "kbd:keyswitch_NumPy_gateon_cherry"
 			(at 44.45 106.68 0)
 			(effects
@@
 			)
 		)
-		(property "Footprint" "kbd:keyswitch_gateron_low_profile_1u"
+		(property "Footprint" "kbd:keyswitch_NumPy_gateon_cherry"
 			(at 135.89 121.92 0)
 			(effects
@@
 			)
 		)
-		(property "Footprint" "kbd:keyswitch_gateron_low_profile_1u"
+		(property "Footprint" "kbd:keyswitch_NumPy_gateon_cherry"
 			(at 158.75 106.68 0)
 			(effects
@@
 			)
 		)
-		(property "Footprint" "kbd:keyswitch_gateron_low_profile_1u"
+		(property "Footprint" "kbd:keyswitch_NumPy_gateon_cherry"
 			(at 158.75 121.92 0)
 			(effects
@@
 			)
 		)
-		(property "Footprint" "kbd:keyswitch_gateron_low_profile_1u"
+		(property "Footprint" "kbd:keyswitch_NumPy_gateon_cherry"
 			(at 101.6 121.92 0)
 			(effects
@@
 			)
 		)
-		(property "Footprint" "kbd:keyswitch_gateron_low_profile_1u"
+		(property "Footprint" "kbd:keyswitch_NumPy_gateon_cherry"
 			(at 55.88 121.92 0)
 			(effects
@@
 			)
 		)
-		(property "Footprint" "kbd:keyswitch_gateron_low_profile_1u"
+		(property "Footprint" "kbd:keyswitch_NumPy_gateon_cherry"
 			(at 90.17 121.92 0)
 			(effects
@@
 			)
 		)
-		(property "Footprint" "kbd:keyswitch_gateron_low_profile_1u"
+		(property "Footprint" "kbd:keyswitch_NumPy_gateon_cherry"
 			(at 44.45 121.92 0)
 			(effects
@@
 			)
 		)
-		(property "Footprint" "kbd:keyswitch_gateron_low_profile_1u"
+		(property "Footprint" "kbd:keyswitch_NumPy_gateon_cherry"
 			(at 55.88 137.16 0)
 			(effects
@@
 			)
 		)
-		(property "Footprint" "kbd:keyswitch_gateron_low_profile_1u"
+		(property "Footprint" "kbd:keyswitch_NumPy_gateon_cherry"
 			(at 67.31 137.16 0)
 			(effects
@@
 			)
 		)
-		(property "Footprint" "kbd:keyswitch_gateron_low_profile_1u"
+		(property "Footprint" "kbd:keyswitch_NumPy_gateon_cherry"
 			(at 33.02 121.92 0)
 			(effects
@@
 			)
 		)
-		(property "Footprint" "kbd:keyswitch_gateron_low_profile_1u"
+		(property "Footprint" "kbd:keyswitch_NumPy_gateon_cherry"
 			(at 158.75 137.16 0)
 			(effects
@@
 			)
 		)
-		(property "Footprint" "kbd:keyswitch_gateron_low_profile_1u"
+		(property "Footprint" "kbd:keyswitch_NumPy_gateon_cherry"
 			(at 101.6 137.16 0)
 			(effects
@@
 			)
 		)
-		(property "Footprint" "kbd:keyswitch_gateron_low_profile_1u"
+		(property "Footprint" "kbd:keyswitch_NumPy_gateon_cherry"
 			(at 124.46 152.4 0)
 			(effects
@@
 			)
 		)
-		(property "Footprint" "kbd:keyswitch_gateron_low_profile_1u"
+		(property "Footprint" "kbd:keyswitch_NumPy_gateon_cherry"
 			(at 44.45 152.4 0)
 			(effects
@@
 			)
 		)
-		(property "Footprint" "kbd:keyswitch_gateron_low_profile_1u"
+		(property "Footprint" "kbd:keyswitch_NumPy_gateon_cherry"
 			(at 101.6 106.68 0)
 			(effects
@@
 			)
 		)
-		(property "Footprint" "kbd:keyswitch_gateron_low_profile_1u"
+		(property "Footprint" "kbd:keyswitch_NumPy_gateon_cherry"
 			(at 113.03 121.92 0)
 			(effects
@@
 			)
 		)
-		(property "Footprint" "kbd:keyswitch_gateron_low_profile_1u"
+		(property "Footprint" "kbd:keyswitch_NumPy_gateon_cherry"
 			(at 67.31 106.68 0)
 			(effects
@@
 			)
 		)
-		(property "Footprint" "kbd:keyswitch_gateron_low_profile_1u"
+		(property "Footprint" "kbd:keyswitch_NumPy_gateon_cherry"
 			(at 101.6 152.4 0)
 			(effects
@@
 			)
 		)
-		(property "Footprint" "kbd:keyswitch_gateron_low_profile_1u"
+		(property "Footprint" "kbd:keyswitch_NumPy_gateon_cherry"
 			(at 90.17 152.4 0)
 			(effects
@@
 			)
 		)
-		(property "Footprint" "kbd:keyswitch_gateron_low_profile_1u"
+		(property "Footprint" "kbd:keyswitch_NumPy_gateon_cherry"
 			(at 78.74 121.92 0)
 			(effects
@@
 			)
 		)
-		(property "Footprint" "kbd:keyswitch_gateron_low_profile_1u"
+		(property "Footprint" "kbd:keyswitch_NumPy_gateon_cherry"
 			(at 135.89 152.4 0)
 			(effects
@@
 			)
 		)
-		(property "Footprint" "kbd:keyswitch_gateron_low_profile_1u"
+		(property "Footprint" "kbd:keyswitch_NumPy_gateon_cherry"
 			(at 67.31 121.92 0)
 			(effects
@@
 			)
 		)
-		(property "Footprint" "kbd:keyswitch_gateron_low_profile_1u"
+		(property "Footprint" "kbd:keyswitch_NumPy_gateon_cherry"
 			(at 135.89 137.16 0)
 			(effects
@@
 			)
 		)
-		(property "Footprint" "kbd:keyswitch_gateron_low_profile_1u"
+		(property "Footprint" "kbd:keyswitch_NumPy_gateon_cherry"
 			(at 135.89 106.68 0)
 			(effects
@@
 			)
 		)
-		(property "Footprint" "kbd:keyswitch_gateron_low_profile_1u"
+		(property "Footprint" "kbd:keyswitch_NumPy_gateon_cherry"
 			(at 33.02 137.16 0)
 			(effects
@@
 			)
 		)
-		(property "Footprint" "kbd:keyswitch_gateron_low_profile_1u"
+		(property "Footprint" "kbd:keyswitch_NumPy_gateon_cherry"
 			(at 67.31 152.4 0)
 			(effects
@@
 			)
 		)
-		(property "Footprint" "kbd:keyswitch_gateron_low_profile_1u"
+		(property "Footprint" "kbd:keyswitch_NumPy_gateon_cherry"
 			(at 78.74 137.16 0)
 			(effects
@@
 			)
 		)
-		(property "Footprint" "kbd:keyswitch_gateron_low_profile_1u"
+		(property "Footprint" "kbd:keyswitch_NumPy_gateon_cherry"
 			(at 78.74 152.4 0)
 			(effects
@@
 			)
 		)
-		(property "Footprint" "kbd:keyswitch_gateron_low_profile_1u"
+		(property "Footprint" "kbd:keyswitch_NumPy_gateon_cherry"
 			(at 78.74 106.68 0)
 			(effects
@@
 			)
 		)
-		(property "Footprint" "kbd:keyswitch_gateron_low_profile_1u"
+		(property "Footprint" "kbd:keyswitch_NumPy_gateon_cherry"
 			(at 147.32 137.16 0)
 			(effects
@@
 			)
 		)
-		(property "Footprint" "kbd:keyswitch_gateron_low_profile_1u"
+		(property "Footprint" "kbd:keyswitch_NumPy_gateon_cherry"
 			(at 147.32 121.92 0)
 			(effects
@@
 			)
 		)
-		(property "Footprint" "kbd:keyswitch_gateron_low_profile_1u"
+		(property "Footprint" "kbd:keyswitch_NumPy_gateon_cherry"
 			(at 90.17 106.68 0)
 			(effects
@@
 			)
 		)
-		(property "Footprint" "kbd:keyswitch_gateron_low_profile_1u"
+		(property "Footprint" "kbd:keyswitch_NumPy_gateon_cherry"
 			(at 113.03 137.16 0)
 			(effects
@@
 			)
 		)
-		(property "Footprint" "kbd:keyswitch_gateron_low_profile_1u"
+		(property "Footprint" "kbd:keyswitch_NumPy_gateon_cherry"
 			(at 33.02 106.68 0)
 			(effects
@@
 			)
 		)
-		(property "Footprint" "kbd:keyswitch_gateron_low_profile_1u"
+		(property "Footprint" "kbd:keyswitch_NumPy_gateon_cherry"
 			(at 113.03 152.4 0)
 			(effects
@@
 			)
 		)
-		(property "Footprint" "kbd:keyswitch_gateron_low_profile_1u"
+		(property "Footprint" "kbd:keyswitch_NumPy_gateon_cherry"
 			(at 124.46 121.92 0)
 			(effects
@@
 			)
 		)
-		(property "Footprint" "kbd:keyswitch_gateron_low_profile_1u"
+		(property "Footprint" "kbd:keyswitch_NumPy_gateon_cherry"
 			(at 124.46 137.16 0)
 			(effects
@@
 			)
 		)
-		(property "Footprint" "kbd:keyswitch_gateron_low_profile_1u"
+		(property "Footprint" "kbd:keyswitch_NumPy_gateon_cherry"
 			(at 33.02 152.4 0)
 			(effects
@@
 			)
 		)
-		(property "Footprint" "kbd:keyswitch_gateron_low_profile_1u"
+		(property "Footprint" "kbd:keyswitch_NumPy_gateon_cherry"
 			(at 147.32 152.4 0)
 			(effects
@@
 			)
 		)
-		(property "Footprint" "kbd:keyswitch_gateron_low_profile_1u"
+		(property "Footprint" "kbd:keyswitch_NumPy_gateon_cherry"
 			(at 55.88 152.4 0)
 			(effects
@@
 			)
 		)
-		(property "Footprint" "kbd:keyswitch_gateron_low_profile_1u"
+		(property "Footprint" "kbd:keyswitch_NumPy_gateon_cherry"
 			(at 44.45 137.16 0)
 			(effects
@@
 			)
 		)
-		(property "Footprint" "kbd:keyswitch_gateron_low_profile_1u"
+		(property "Footprint" "kbd:keyswitch_NumPy_gateon_cherry"
 			(at 147.32 106.68 0)
 			(effects
@@
 			)
 		)
-		(property "Footprint" "kbd:keyswitch_gateron_low_profile_1u"
+		(property "Footprint" "kbd:keyswitch_NumPy_gateon_cherry"
 			(at 124.46 106.68 0)
 			(effects
@@
 			)
 		)
-		(property "Footprint" "kbd:keyswitch_gateron_low_profile_1u"
+		(property "Footprint" "kbd:keyswitch_NumPy_gateon_cherry"
 			(at 113.03 106.68 0)
 			(effects
@@
 			)
 		)
-		(property "Footprint" "kbd:keyswitch_gateron_low_profile_1u"
+		(property "Footprint" "kbd:keyswitch_NumPy_gateon_cherry"
 			(at 90.17 137.16 0)
 			(effects

Commit message: Продолжаем. Натянули. Расставляем
Parts:
- K1, K10, K11, K12, K13, K14, K15, K16, K17, K18, K19, K2, K20, K21, K22, K23, K24, K25, K26, K27, K28, K29, K3, K30, K31, K32, K33, K34, K35, K36, K37, K38, K39, K4, K40, K41, K42, K43, K44, K45, K46, K47, K48, K5, K6, K7, K8, K9: footprint kbd:keyswitch_NumPy_gateon_cherry -> kbd:SW_Gateron_LowProfile_THT
Changed lines of the file:
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@@
 			)
 		)
-		(property "Footprint" "kbd:keyswitch_NumPy_gateon_cherry"
+		(property "Footprint" "kbd:SW_Gateron_LowProfile_THT"
 			(at 158.75 152.4 0)
 			(effects
@@
 			)
 		)
-		(property "Footprint" "kbd:keyswitch_NumPy_gateon_cherry"
+		(property "Footprint" "kbd:SW_Gateron_LowProfile_THT"
 			(at 55.88 106.68 0)
 			(effects
@@
 			)
 		)
-		(property "Footprint" "kbd:keyswitch_NumPy_gateon_cherry"
+		(property "Footprint" "kbd:SW_Gateron_LowProfile_THT"
 			(at 44.45 106.68 0)
 			(effects
@@
 			)
 		)
-		(property "Footprint" "kbd:keyswitch_NumPy_gateon_cherry"
+		(property "Footprint" "kbd:SW_Gateron_LowProfile_THT"
 			(at 135.89 121.92 0)
 			(effects
@@
 			)
 		)
-		(property "Footprint" "kbd:keyswitch_NumPy_gateon_cherry"
+		(property "Footprint" "kbd:SW_Gateron_LowProfile_THT"
 			(at 158.75 106.68 0)
 			(effects
@@
 			)
 		)
-		(property "Footprint" "kbd:keyswitch_NumPy_gateon_cherry"
+		(property "Footprint" "kbd:SW_Gateron_LowProfile_THT"
 			(at 158.75 121.92 0)
 			(effects
@@
 			)
 		)
-		(property "Footprint" "kbd:keyswitch_NumPy_gateon_cherry"
+		(property "Footprint" "kbd:SW_Gateron_LowProfile_THT"
 			(at 101.6 121.92 0)
 			(effects
@@
 			)
 		)
-		(property "Footprint" "kbd:keyswitch_NumPy_gateon_cherry"
+		(property "Footprint" "kbd:SW_Gateron_LowProfile_THT"
 			(at 55.88 121.92 0)
 			(effects
@@
 			)
 		)
-		(property "Footprint" "kbd:keyswitch_NumPy_gateon_cherry"
+		(property "Footprint" "kbd:SW_Gateron_LowProfile_THT"
 			(at 90.17 121.92 0)
 			(effects
@@
 			)
 		)
-		(property "Footprint" "kbd:keyswitch_NumPy_gateon_cherry"
+		(property "Footprint" "kbd:SW_Gateron_LowProfile_THT"
 			(at 44.45 121.92 0)
 			(effects
@@
 			)
 		)
-		(property "Footprint" "kbd:keyswitch_NumPy_gateon_cherry"
+		(property "Footprint" "kbd:SW_Gateron_LowProfile_THT"
 			(at 55.88 137.16 0)
 			(effects
@@
 			)
 		)
-		(property "Footprint" "kbd:keyswitch_NumPy_gateon_cherry"
+		(property "Footprint" "kbd:SW_Gateron_LowProfile_THT"
 			(at 67.31 137.16 0)
 			(effects
@@
 			)
 		)
-		(property "Footprint" "kbd:keyswitch_NumPy_gateon_cherry"
+		(property "Footprint" "kbd:SW_Gateron_LowProfile_THT"
 			(at 33.02 121.92 0)
 			(effects
@@
 			)
 		)
-		(property "Footprint" "kbd:keyswitch_NumPy_gateon_cherry"
+		(property "Footprint" "kbd:SW_Gateron_LowProfile_THT"
 			(at 158.75 137.16 0)
 			(effects
@@
 			)
 		)
-		(property "Footprint" "kbd:keyswitch_NumPy_gateon_cherry"
+		(property "Footprint" "kbd:SW_Gateron_LowProfile_THT"
 			(at 101.6 137.16 0)
 			(effects
@@
 			)
 		)
-		(property "Footprint" "kbd:keyswitch_NumPy_gateon_cherry"
+		(property "Footprint" "kbd:SW_Gateron_LowProfile_THT"
 			(at 124.46 152.4 0)
 			(effects
@@
 			)
 		)
-		(property "Footprint" "kbd:keyswitch_NumPy_gateon_cherry"
+		(property "Footprint" "kbd:SW_Gateron_LowProfile_THT"
 			(at 44.45 152.4 0)
 			(effects
@@
 			)
 		)
-		(property "Footprint" "kbd:keyswitch_NumPy_gateon_cherry"
+		(property "Footprint" "kbd:SW_Gateron_LowProfile_THT"
 			(at 101.6 106.68 0)
 			(effects
@@
 			)
 		)
-		(property "Footprint" "kbd:keyswitch_NumPy_gateon_cherry"
+		(property "Footprint" "kbd:SW_Gateron_LowProfile_THT"
 			(at 113.03 121.92 0)
 			(effects
@@
 			)
 		)
-		(property "Footprint" "kbd:keyswitch_NumPy_gateon_cherry"
+		(property "Footprint" "kbd:SW_Gateron_LowProfile_THT"
 			(at 67.31 106.68 0)
 			(effects
@@
 			)
 		)
-		(property "Footprint" "kbd:keyswitch_NumPy_gateon_cherry"
+		(property "Footprint" "kbd:SW_Gateron_LowProfile_THT"
 			(at 101.6 152.4 0)
 			(effects
@@
 			)
 		)
-		(property "Footprint" "kbd:keyswitch_NumPy_gateon_cherry"
+		(property "Footprint" "kbd:SW_Gateron_LowProfile_THT"
 			(at 90.17 152.4 0)
 			(effects
@@
 			)
 		)
-		(property "Footprint" "kbd:keyswitch_NumPy_gateon_cherry"
+		(property "Footprint" "kbd:SW_Gateron_LowProfile_THT"
 			(at 78.74 121.92 0)
 			(effects
@@
 			)
 		)
-		(property "Footprint" "kbd:keyswitch_NumPy_gateon_cherry"
+		(property "Footprint" "kbd:SW_Gateron_LowProfile_THT"
 			(at 135.89 152.4 0)
 			(effects
@@
 			)
 		)
-		(property "Footprint" "kbd:keyswitch_NumPy_gateon_cherry"
+		(property "Footprint" "kbd:SW_Gateron_LowProfile_THT"
 			(at 67.31 121.92 0)
 			(effects
@@
 			)
 		)
-		(property "Footprint" "kbd:keyswitch_NumPy_gateon_cherry"
+		(property "Footprint" "kbd:SW_Gateron_LowProfile_THT"
 			(at 135.89 137.16 0)
 			(effects
@@
 			)
 		)
-		(property "Footprint" "kbd:keyswitch_NumPy_gateon_cherry"
+		(property "Footprint" "kbd:SW_Gateron_LowProfile_THT"
 			(at 135.89 106.68 0)
 			(effects
@@
 			)
 		)
-		(property "Footprint" "kbd:keyswitch_NumPy_gateon_cherry"
+		(property "Footprint" "kbd:SW_Gateron_LowProfile_THT"
 			(at 33.02 137.16 0)
 			(effects
@@
 			)
 		)
-		(property "Footprint" "kbd:keyswitch_NumPy_gateon_cherry"
+		(property "Footprint" "kbd:SW_Gateron_LowProfile_THT"
 			(at 67.31 152.4 0)
 			(effects
@@
 			)
 		)
-		(property "Footprint" "kbd:keyswitch_NumPy_gateon_cherry"
+		(property "Footprint" "kbd:SW_Gateron_LowProfile_THT"
 			(at 78.74 137.16 0)
 			(effects
@@
 			)
 		)
-		(property "Footprint" "kbd:keyswitch_NumPy_gateon_cherry"
+		(property "Footprint" "kbd:SW_Gateron_LowProfile_THT"
 			(at 78.74 152.4 0)
 			(effects
@@
 			)
 		)
-		(property "Footprint" "kbd:keyswitch_NumPy_gateon_cherry"
+		(property "Footprint" "kbd:SW_Gateron_LowProfile_THT"
 			(at 78.74 106.68 0)
 			(effects
@@
 			)
 		)
-		(property "Footprint" "kbd:keyswitch_NumPy_gateon_cherry"
+		(property "Footprint" "kbd:SW_Gateron_LowProfile_THT"
 			(at 147.32 137.16 0)
 			(effects
@@
 			)
 		)
-		(property "Footprint" "kbd:keyswitch_NumPy_gateon_cherry"
+		(property "Footprint" "kbd:SW_Gateron_LowProfile_THT"
 			(at 147.32 121.92 0)
 			(effects
@@
 			)
 		)
-		(property "Footprint" "kbd:keyswitch_NumPy_gateon_cherry"
+		(property "Footprint" "kbd:SW_Gateron_LowProfile_THT"
 			(at 90.17 106.68 0)
 			(effects
@@
 			)
 		)
-		(property "Footprint" "kbd:keyswitch_NumPy_gateon_cherry"
+		(property "Footprint" "kbd:SW_Gateron_LowProfile_THT"
 			(at 113.03 137.16 0)
 			(effects
@@
 			)
 		)
-		(property "Footprint" "kbd:keyswitch_NumPy_gateon_cherry"
+		(property "Footprint" "kbd:SW_Gateron_LowProfile_THT"
 			(at 33.02 106.68 0)
 			(effects
@@
 			)
 		)
-		(property "Footprint" "kbd:keyswitch_NumPy_gateon_cherry"
+		(property "Footprint" "kbd:SW_Gateron_LowProfile_THT"
 			(at 113.03 152.4 0)
 			(effects
@@
 			)
 		)
-		(property "Footprint" "kbd:keyswitch_NumPy_gateon_cherry"
+		(property "Footprint" "kbd:SW_Gateron_LowProfile_THT"
 			(at 124.46 121.92 0)
 			(effects
@@
 			)
 		)
-		(property "Footprint" "kbd:keyswitch_NumPy_gateon_cherry"
+		(property "Footprint" "kbd:SW_Gateron_LowProfile_THT"
 			(at 124.46 137.16 0)
 			(effects
@@
 			)
 		)
-		(property "Footprint" "kbd:keyswitch_NumPy_gateon_cherry"
+		(property "Footprint" "kbd:SW_Gateron_LowProfile_THT"
 			(at 33.02 152.4 0)
 			(effects
@@
 			)
 		)
-		(property "Footprint" "kbd:keyswitch_NumPy_gateon_cherry"
+		(property "Footprint" "kbd:SW_Gateron_LowProfile_THT"
 			(at 147.32 152.4 0)
 			(effects
@@
 			)
 		)
-		(property "Footprint" "kbd:keyswitch_NumPy_gateon_cherry"
+		(property "Footprint" "kbd:SW_Gateron_LowProfile_THT"
 			(at 55.88 152.4 0)
 			(effects
@@
 			)
 		)
-		(property "Footprint" "kbd:keyswitch_NumPy_gateon_cherry"
+		(property "Footprint" "kbd:SW_Gateron_LowProfile_THT"
 			(at 44.45 137.16 0)
 			(effects
@@
 			)
 		)
-		(property "Footprint" "kbd:keyswitch_NumPy_gateon_cherry"
+		(property "Footprint" "kbd:SW_Gateron_LowProfile_THT"
 			(at 147.32 106.68 0)
 			(effects
@@
 			)
 		)
-		(property "Footprint" "kbd:keyswitch_NumPy_gateon_cherry"
+		(property "Footprint" "kbd:SW_Gateron_LowProfile_THT"
 			(at 124.46 106.68 0)
 			(effects
@@
 			)
 		)
-		(property "Footprint" "kbd:keyswitch_NumPy_gateon_cherry"
+		(property "Footprint" "kbd:SW_Gateron_LowProfile_THT"
 			(at 113.03 106.68 0)
 			(effects
@@
 			)
 		)
-		(property "Footprint" "kbd:keyswitch_NumPy_gateon_cherry"
+		(property "Footprint" "kbd:SW_Gateron_LowProfile_THT"
 			(at 90.17 137.16 0)
 			(effects
