File: keyvas.kicad_sch (KiCad schematic)
At the start: 130 parts, among them J2 SWD, J3 USB-C Conn, J4 Conn_01x02_Female, K1 KEYSW, K10 KEYSW, K11 KEYSW, K12 KEYSW, K13 KEYSW, K14 KEYSW, K15 KEYSW, K16 KEYSW, K17 KEYSW, K18 KEYSW, K19 KEYSW, K2 KEYSW, K20 KEYSW, K21 KEYSW, K22 KEYSW, K23 KEYSW, K24 KEYSW, K25 KEYSW, K26 KEYSW, K27 KEYSW, K28 KEYSW, K29 KEYSW, K3 KEYSW, K30 KEYSW, K31 KEYSW, K32 KEYSW, K33 KEYSW, K34 KEYSW, K35 KEYSW, K36 KEYSW, K37 KEYSW, K38 KEYSW, K39 KEYSW, K4 KEYSW, K40 KEYSW, K41 KEYSW, K42 KEYSW, K43 KEYSW, K44 KEYSW, K45 KEYSW, K46 KEYSW, K47 KEYSW, K48 KEYSW, K5 KEYSW, K6 KEYSW, K7 KEYSW, K8 KEYSW, K9 KEYSW, Q2 AO3407, SW31 SW_SPDT, U2 XC6220B331MR-G, U3 TP4054, U4 USBLC6-2SC6, U5 E73-2G4M08S1C, X1 32.768kHz

Commit message: Двигаем далее
Parts:
- added H2, H7, H8: MountingHole, kbd:Hole 3,2, symbol Mechanical:MountingHole
- H1, H3, H4, H5, H6: footprint kbd:M2-MountingHole-Standoff -> kbd:Hole 3,2
- J3: footprint kbd:USB-C_C168688_REV -> kbd:TYPE-C-31-M-13C
- U5: footprint E73-2G4M08S1C:E73-2G4M08S1C -> E73-2G4M08S1C-master:E73-2G4M08S1C-52840
Changed lines of the file:
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@@
 			)
 		)
-		(property "Footprint" "E73-2G4M08S1C:E73-2G4M08S1C"
+		(property "Footprint" "E73-2G4M08S1C-master:E73-2G4M08S1C-52840"
 			(at 46.99 60.706 0)
 			(effects
@@
 			)
 		)
-		(property "Footprint" "kbd:M2-MountingHole-Standoff"
+		(property "Footprint" "kbd:Hole 3,2"
 			(at 201.93 97.79 0)
 			(effects
@@
 			)
 		)
-		(property "Footprint" "kbd:M2-MountingHole-Standoff"
+		(property "Footprint" "kbd:Hole 3,2"
 			(at 201.93 87.63 0)
 			(effects
@@
 	)
 	(symbol
+		(lib_name "MountingHole_1")
+		(lib_id "Mechanical:MountingHole")
+		(at 201.93 107.95 0)
+		(unit 1)
+		(exclude_from_sim no)
+		(in_bom yes)
+		(on_board yes)
+		(dnp no)
+		(property "Reference" "H2"
+			(at 205.74 106.426 0)
+			(effects
+				(font
+					(size 1.27 1.27)
+				)
+				(justify left)
+			)
+		)
+		(property "Value" "MountingHole"
+			(at 205.74 108.966 0)
+			(effects
+				(font
+					(size 1.27 1.27)
+				)
+				(justify left)
+			)
+		)
+		(property "Footprint" "kbd:Hole 3,2"
+			(at 201.93 107.95 0)
+			(effects
+				(font
+					(size 1.27 1.27)
+				)
+				(hide yes)
+			)
+		)
+		(property "Datasheet" "~"
+			(at 201.93 107.95 0)
+			(effects
+				(font
+					(size 1.27 1.27)
+				)
+				(hide yes)
+			)
+		)
+		(property "Description" "Mounting Hole without connection"
+			(at 201.93 107.95 0)
+			(effects
+				(font
+					(size 1.27 1.27)
+				)
+				(hide yes)
+			)
+		)
+		(instances
+			(project ""
+				(path "/3b17620c-a565-4e9f-bd7f-b6a9b37841e9"
+					(reference "H2")
+					(unit 1)
+				)
+			)
+		)
+	)
+	(symbol
 		(lib_id "Keyboard_Components:KEYSW")
 		(at 158.75 142.24 0)
@@
 			)
 		)
-		(property "Footprint" "kbd:M2-MountingHole-Standoff"
+		(property "Footprint" "kbd:Hole 3,2"
 			(at 201.93 82.55 0)
 			(effects
@@
 	)
 	(symbol
+		(lib_name "KEYSW_1")
 		(lib_id "Keyboard_Components:KEYSW")
 		(at 101.6 142.24 0)
@@
 			)
 		)
-		(property "Footprint" "kbd:USB-C_C168688_REV"
+		(property "Footprint" "kbd:TYPE-C-31-M-13C"
 			(at 171.6278 17.145 0)
 			(effects
@@
 	)
 	(symbol
+		(lib_name "MountingHole_2")
+		(lib_id "Mechanical:MountingHole")
+		(at 201.93 113.03 0)
+		(unit 1)
+		(exclude_from_sim no)
+		(in_bom yes)
+		(on_board yes)
+		(dnp no)
+		(property "Reference" "H7"
+			(at 205.74 111.76 0)
+			(effects
+				(font
+					(size 1.27 1.27)
+				)
+				(justify left)
+			)
+		)
+		(property "Value" "MountingHole"
+			(at 205.74 114.3 0)
+			(effects
+				(font
+					(size 1.27 1.27)
+				)
+				(justify left)
+			)
+		)
+		(property "Footprint" "kbd:Hole 3,2"
+			(at 201.93 113.03 0)
+			(effects
+				(font
+					(size 1.27 1.27)
+				)
+				(hide yes)
+			)
+		)
+		(property "Datasheet" "~"
+			(at 201.93 113.03 0)
+			(effects
+				(font
+					(size 1.27 1.27)
+				)
+				(hide yes)
+			)
+		)
+		(property "Description" "Mounting Hole without connection"
+			(at 201.93 113.03 0)
+			(effects
+				(font
+					(size 1.27 1.27)
+				)
+				(hide yes)
+			)
+		)
+		(instances
+			(project ""
+				(path "/3b17620c-a565-4e9f-bd7f-b6a9b37841e9"
+					(reference "H7")
+					(unit 1)
+				)
+			)
+		)
+	)
+	(symbol
 		(lib_id "Mechanical:MountingHole")
 		(at 201.93 102.87 0)
@@
 			)
 		)
-		(property "Footprint" "kbd:M2-MountingHole-Standoff"
+		(property "Footprint" "kbd:Hole 3,2"
 			(at 201.93 102.87 0)
 			(effects
@@
 			)
 		)
-		(property "Footprint" "kbd:M2-MountingHole-Standoff"
+		(property "Footprint" "kbd:Hole 3,2"
 			(at 201.93 92.71 0)
 			(effects
@@
 					(unit 1)
 				)
+			)
+		)
+	)
+	(symbol
+		(lib_name "MountingHole_2")
+		(lib_id "Mechanical:MountingHole")
+		(at 201.93 118.11 0)
+		(unit 1)
+		(exclude_from_sim no)
+		(in_bom yes)
+		(on_board yes)
+		(dnp no)
+		(property "Reference" "H8"
+			(at 205.74 116.84 0)
+			(effects
+				(font
+					(size 1.27 1.27)
+				)
+				(justify left)
+			)
+		)
+		(property "Value" "MountingHole"
+			(at 205.74 119.38 0)
+			(effects
+				(font
+					(size 1.27 1.27)
+				)
+				(justify left)
+			)
+		)
+		(property "Footprint" "kbd:Hole 3,2"
+			(at 201.93 118.11 0)
+			(effects
+				(font
+					(size 1.27 1.27)
+				)
+				(hide yes)
+			)
+		)
+		(property "Datasheet" "~"
+			(at 201.93 118.11 0)
+			(effects
+				(font
+					(size 1.27 1.27)
+				)
+				(hide yes)
+			)
+		)
+		(property "Description" "Mounting Hole without connection"
+			(at 201.93 118.11 0)
+			(effects
+				(font
+					(size 1.27 1.27)
+				)
+				(hide yes)
+			)
+		)
+		(instances
+			(project "keyvas"
+				(path "/3b17620c-a565-4e9f-bd7f-b6a9b37841e9"
+					(reference "H8")
+					(unit 1)
+				)

Commit message: Двигаем далее 2
Connections:
- net BATTERY_PIN: now also U5.35 (P0.24); no longer U5.7 (P0.02/AIN0*)
- net BLUE_LED: now also U5.33 (P0.13); no longer U5.2 (P1.10*)
- net COL0: now also U5.42 (P1.06*); no longer U5.10 (P0.30/AIN6*)
- net COL1: now also U5.40 (P1.04*); no longer U5.9 (P0.31/AIN7*)
- net COL10: now also U5.18 (P0.04/AIN2); no longer U5.16 (P0.08)
- net COL11: now also U5.16 (P0.08); no longer U5.14 (P0.06)
- net COL2: now also U5.38 (P1.02*); no longer U5.8 (P0.29/AIN5*)
- net COL3: now also U5.36 (P1.00); no longer U5.6 (P1.13*)
- net COL4: now also U5.34 (P0.22); no longer U5.4 (P0.28/AIN4*)
- net COL5: now also U5.32 (P0.20); no longer U5.3 (P0.03/AIN1*)
- net COL6: now also U5.30 (P0.17); no longer U5.1 (P1.11*)
- net COL7: now also U5.28 (P0.15); no longer U5.22 (P0.07)
- net COL8: now also U5.22 (P0.07); no longer U5.20 (P0.12)
- net COL9: now also U5.20 (P0.12); no longer U5.18 (P0.04/AIN2)
- net ROW0: now also U5.1 (P1.11*); no longer U5.43 (P0.10/NFC2*)
- net ROW1: now also U5.2 (P1.10*); no longer U5.28 (P0.15)
- net ROW2: now also U5.3 (P0.03/AIN1*); no longer U5.33 (P0.13)
- net ROW3: now also U5.4 (P0.28/AIN4*); no longer U5.35 (P0.24)

Commit message: finish 2
Connections:
- net ENCBTN: now reaches U5.6 (P1.13*)
- net ENC2: now reaches U5.7 (P0.02/AIN0*)
- net ENC1: now reaches U5.8 (P0.29/AIN5*)
Changed lines of the file:
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@@
 	(wire
 		(pts
+			(xy 114.3 58.42) (xy 118.11 58.42)
+		)
+		(stroke
+			(width 0)
+			(type default)
+		)
+	)
+	(wire
+		(pts
 			(xy 83.82 111.76) (xy 83.82 127)
 		)
@@
 	(wire
 		(pts
+			(xy 114.3 54.61) (xy 118.11 54.61)
+		)
+		(stroke
+			(width 0)
+			(type default)
+		)
+	)
+	(wire
+		(pts
 			(xy 92.71 25.4) (xy 92.71 26.67)
 		)
@@
 	(wire
 		(pts
+			(xy 114.3 50.8) (xy 118.11 50.8)
+		)
+		(stroke
+			(width 0)
+			(type default)
+		)
+	)
+	(wire
+		(pts
 			(xy 249.555 52.07) (xy 249.555 49.53)
 		)
@@
 		)
 	)
+	(global_label "ENCBTN"
+		(shape input)
+		(at 118.11 58.42 0)
+		(fields_autoplaced yes)
+		(effects
+			(font
+				(size 1.27 1.27)
+			)
+			(justify left)
+		)
+		(property "Intersheetrefs" "${INTERSHEET_REFS}"
+			(at 128.4128 58.42 0)
+			(effects
+				(font
+					(size 1.27 1.27)
+				)
+				(justify left)
+				(hide yes)
+			)
+		)
+	)
 	(global_label "USBN"
 		(shape input)
@@
 		)
 	)
+	(global_label "ENC2"
+		(shape input)
+		(at 118.11 54.61 0)
+		(fields_autoplaced yes)
+		(effects
+			(font
+				(size 1.27 1.27)
+			)
+			(justify left)
+		)
+		(property "Intersheetrefs" "${INTERSHEET_REFS}"
+			(at 126.0542 54.61 0)
+			(effects
+				(font
+					(size 1.27 1.27)
+				)
+				(justify left)
+				(hide yes)
+			)
+		)
+	)
 	(global_label "COL6"
 		(shape input)
@@
 				(hide yes)
 			)
+		)
+	)
+	(global_label "ENC1"
+		(shape input)
+		(at 118.11 50.8 0)
+		(fields_autoplaced yes)
+		(effects
+			(font
+				(size 1.27 1.27)
+			)
+			(justify left)
+		)
+		(property "Intersheetrefs" "${INTERSHEET_REFS}"
+			(at 126.0542 50.8 0)
+			(effects
+				(font
+					(size 1.27 1.27)
+				)
+				(justify left)
+				(hide yes)
+			)
