File: keyvas.kicad_pcb (KiCad board)
At the start: 2 copper layers, 130 parts, among them J2 SWD, J3 USB-C Conn, J4 Conn_01x02_Female, K1 KEYSW, K10 KEYSW, K11 KEYSW, K12 KEYSW, K13 KEYSW, K14 KEYSW, K15 KEYSW, K16 KEYSW, K17 KEYSW, K18 KEYSW, K19 KEYSW, K2 KEYSW, K20 KEYSW, K21 KEYSW, K22 KEYSW, K23 KEYSW, K24 KEYSW, K25 KEYSW, K26 KEYSW, K27 KEYSW, K28 KEYSW, K29 KEYSW, K3 KEYSW, K30 KEYSW, K31 KEYSW, K32 KEYSW, K33 KEYSW, K34 KEYSW, K35 KEYSW, K36 KEYSW, K37 KEYSW, K38 KEYSW, K39 KEYSW, K4 KEYSW, K40 KEYSW, K41 KEYSW, K42 KEYSW, K43 KEYSW, K44 KEYSW, K45 KEYSW, K46 KEYSW, K47 KEYSW, K48 KEYSW, K5 KEYSW, K6 KEYSW, K7 KEYSW, K8 KEYSW, K9 KEYSW, Q2 AO3407, SW31 SW_SPDT, U2 XC6220B331MR-G, U3 TP4054, U4 USBLC6-2SC6, U5 E73-2G4M08S1C, X1 32.768kHz

Commit message: fix
Parts:
- moved SW31 218.7 mm to (45.0, 30.0), turned to 180 degrees
- moved U3 215.9 mm to (188.3, 68.0)
- moved RSW1 206.2 mm to (54.3, 30.3), turned to 180 degrees
- moved U2 203.6 mm to (169.8, 67.5)
- moved U4 182.6 mm to (152.7, 67.5)
- moved Q2 173.1 mm to (133.5, 67.5)
- moved U5 105.2 mm to (148.8, 49.9), turned to 180 degrees
- moved J2 6.09 mm to (71.6, 242.8)
- moved J3 3.54 mm to (149.0, 28.0)
- turned K18 to -90 degrees
- turned K19 to 90 degrees
Other:
- board outline added: 228 x 78 mm

Commit message: fix 2
Parts:
- K44: footprint kbd:MX_Alps_Hitek_725_1.5U_reversible -> kbd:keyswitch_gateron_low_profile_1u
- moved H3 223.7 mm to (206.0, 69.4)
- moved H4 223.7 mm to (206.0, 74.4)
- moved H5 223.7 mm to (206.0, 79.4)
- moved H6 223.7 mm to (206.0, 84.4)
- moved J4 200.6 mm to (92.6, 31.3), turned to -90 degrees
- moved J2 182.1 mm to (52.4, 61.7)
- moved D31 182.1 mm to (92.4, 71.8)
- moved D36 182.1 mm to (91.9, 69.0)
- moved F1 182.1 mm to (92.7, 63.5)
- moved X1 182.1 mm to (92.0, 74.7)
- moved R2 171.6 mm to (168.2, 82.2)
- moved R3 171.6 mm to (168.2, 84.7)
- moved R4 171.6 mm to (168.2, 87.2)
- moved R5 171.6 mm to (168.2, 89.7)
- moved R6 171.6 mm to (168.2, 92.2)
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
Commit message: fix 3
Parts:
- added ?: , , F.Cu at (187.0, 49.0)
- added ?: , , F.Cu at (129.8, 75.5)
- added ?: , , F.Cu at (187.0, 87.0)
- moved H5 155.0 mm to (54.0, 49.0)
- moved H4 80.1 mm to (130.0, 49.0)
- moved D36 65.6 mm to (146.8, 105.0)
- moved D35 61.7 mm to (151.3, 105.0)
- moved H3 42.9 mm to (244.0, 49.5)
- moved H6 38.1 mm to (244.0, 87.0)
- moved D31 18.5 mm to (74.2, 68.0)
- moved D45 8.22 mm to (135.5, 105.0)
- moved D40 5.22 mm to (53.0, 102.0), turned to 90 degrees
- moved D41 5.00 mm to (72.0, 102.0), turned to 90 degrees
- moved D42 5.00 mm to (91.0, 102.0), turned to 90 degrees
- moved H1 1.21 mm to (54.0, 87.0)
Routing:
- net COL0: track 0.00 -> 64.8 mm
- net ROW3: track 0.00 -> 38.4 mm
- net Net-(D42-A): track 0.00 -> 4.34 mm
- net Net-(D41-A): track 0.00 -> 4.34 mm
- net Net-(D40-A): track 0.00 -> 4.22 mm
