File: keyvas.kicad_pcb (KiCad board)
At the start: 2 copper layers, 228 x 78 mm, 130 parts, among them J2 SWD, J3 USB-C Conn, J4 Conn_01x02_Female, K1 KEYSW, K10 KEYSW, K11 KEYSW, K12 KEYSW, K13 KEYSW, K14 KEYSW, K15 KEYSW, K16 KEYSW, K17 KEYSW, K18 KEYSW, K19 KEYSW, K2 KEYSW, K20 KEYSW, K21 KEYSW, K22 KEYSW, K23 KEYSW, K24 KEYSW, K25 KEYSW, K26 KEYSW, K27 KEYSW, K28 KEYSW, K29 KEYSW, K3 KEYSW, K30 KEYSW, K31 KEYSW, K32 KEYSW, K33 KEYSW, K34 KEYSW, K35 KEYSW, K36 KEYSW, K37 KEYSW, K38 KEYSW, K39 KEYSW, K4 KEYSW, K40 KEYSW, K41 KEYSW, K42 KEYSW, K43 KEYSW, K44 KEYSW, K45 KEYSW, K46 KEYSW, K47 KEYSW, K48 KEYSW, K5 KEYSW, K6 KEYSW, K7 KEYSW, K8 KEYSW, K9 KEYSW, Q2 AO3407, SW31 SW_SPDT, U2 XC6220B331MR-G, U3 TP4054, U4 USBLC6-2SC6, U5 E73-2G4M08S1C, X1 32.768kHz

Commit message: Продолжаем натягивать сову на глобус
Parts:
- K1, K10, K11, K12, K13, K14, K15, K16, K17, K18, K19, K2, K20, K21, K22, K23, K24, K25, K26, K27, K28, K29, K3, K30, K31, K32, K33, K34, K35, K36, K37, K38, K39, K4, K40, K41, K42, K43, K44, K45, K46, K47, K48, K5, K6, K7, K8, K9: footprint kbd:keyswitch_gateron_low_profile_1u -> kbd:keyswitch_NumPy_gateon_cherry
- moved RSW1 0.08 mm to (54.3, 30.2)
- turned K18 to 90 degrees
- turned K19 to -90 degrees
- turned K6 to 90 degrees
- turned K7 to -90 degrees
Connections:
- U5 pad 12: ROW0 -> unconnected-(U5-P0.26-Pad12)
- U5 pad 30: ROW2 -> unconnected-(U5-P0.17-Pad30)
- U5 pad 32: ROW3 -> unconnected-(U5-P0.20-Pad32)
- U5 pad 33: unconnected-(U5-P0.13-Pad33) -> ROW2
- U5 pad 35: unconnected-(U5-P0.24-Pad35) -> ROW3
- U5 pad 43: unconnected-(U5-P0.10/NFC2*-Pad43) -> ROW0
Other:
- outline, holes or cut-outs redrawn

Commit message: Продолжаем. Натянули. Расставляем
Parts:
- K1, K10, K11, K12, K13, K14, K15, K16, K17, K18, K19, K2, K20, K21, K22, K23, K24, K25, K26, K27, K28, K29, K3, K30, K31, K32, K33, K34, K35, K36, K37, K38, K39, K4, K40, K41, K42, K43, K44, K45, K46, K47, K48, K5, K6, K7, K8, K9: footprint kbd:keyswitch_NumPy_gateon_cherry -> kbd:SW_Gateron_LowProfile_THT
- moved R6 31.4 mm to (166.5, 123.5)
- moved R2 31.4 mm to (166.5, 113.5)
- moved R3 31.4 mm to (166.5, 116.0)
- moved R4 31.4 mm to (166.5, 118.5)
- moved R5 31.4 mm to (166.5, 121.0)
- moved H1 29.7 mm to (25.5, 85.5)
- moved C3 29.6 mm to (129.0, 117.5)
- moved C1 29.6 mm to (129.0, 112.5)
- moved C2 29.6 mm to (129.0, 115.0)
- moved C4 29.6 mm to (129.0, 120.0)
- moved C5 29.6 mm to (129.0, 122.5)
- moved K48 27.4 mm to (226.1, 96.5)
- moved D51 26.9 mm to (234.3, 91.8), turned to -90 degrees
- moved D50 25.0 mm to (217.8, 91.8), turned to -90 degrees
- moved K47 24.9 mm to (209.6, 96.5)
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Routing:
- net ROW0: track 0.00 -> 19.5 mm
- net Net-(D40-A): track 0.00 -> 1.33 mm
Other:
- board outline removed
