File: keyvas.kicad_pcb (KiCad board)
At the start: 2 copper layers, 219.4 x 78 mm, 137 parts, among them J2 SWD, J3 USB-C Conn, J4 Conn_01x02_Female, K1 KEYSW, K10 KEYSW, K11 KEYSW, K12 KEYSW, K13 KEYSW, K14 KEYSW, K15 KEYSW, K16 KEYSW, K17 KEYSW, K18 KEYSW, K19 KEYSW, K2 KEYSW, K20 KEYSW, K21 KEYSW, K22 KEYSW, K23 KEYSW, K24 KEYSW, K25 KEYSW, K26 KEYSW, K27 KEYSW, K28 KEYSW, K29 KEYSW, K3 KEYSW, K30 KEYSW, K31 KEYSW, K32 KEYSW, K33 KEYSW, K34 KEYSW, K35 KEYSW, K36 KEYSW, K37 KEYSW, K38 KEYSW, K39 KEYSW, K4 KEYSW, K40 KEYSW, K41 KEYSW, K42 KEYSW, K43 KEYSW, K44 KEYSW, K45 KEYSW, K46 KEYSW, K47 KEYSW, K48 KEYSW, K5 KEYSW, K6 KEYSW, K7 KEYSW, K8 KEYSW, K9 KEYSW, Q2 AO3407, SW31 SW_SPDT, U2 XC6220B331MR-G, U3 TP4054, U4 USBLC6-2SC6, U5 E73-2G4M08S1C, X1 32.768kHz

Commit message: start case
Routing:
- net USBP: track 178.9 -> 183.2 mm, vias 7 -> 8
- net USBN: track 183.2 -> 178.9 mm, vias 8 -> 7
- added copper zone on B.Cu, net GND
- added copper zone on F.Cu, net GND
